File: EGK_kredsløb.kicad_pcb (KiCad board)
At the start: 2 copper layers, 100 x 70 mm, 50 parts, among them J101 10118194-0001LF, J102 Conn_01x03, J103 Conn_01x06_Pin, J104 Conn_01x03, J107 Conn_01x03, J108 Mini_Jack_5pins, J110 Conn_01x06_Pin, J111 Conn_01x06_Pin, J112 Conn_01x06_Pin, J113 Conn_01x06_Pin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

Commit message: opstart af routing
Parts:
- moved C109 0.50 mm to (139.0, 99.0)
Routing:
- net /VGND: track 0.00 -> 134.2 mm
- net /R_ARM: track 2.54 -> 43.4 mm
- net /R_LEG: track 0.00 -> 31.0 mm
- net /HP+: track 0.00 -> 29.4 mm
- net /L_ARM: track 0.00 -> 25.7 mm
- net /GAIN_BLOCK_OUT: track 0.00 -> 16.1 mm
- net Net-(R112-Pad1): track 0.00 -> 16.1 mm
- net /V_BIAS: track 0.00 -> 15.7 mm
- net /ADC_IN: track 0.00 -> 14.1 mm
- net /HP_OUT: track 0.00 -> 10.3 mm
- net Net-(C101-Pad1): track 0.00 -> 9.11 mm
- net /LP+: track 0.00 -> 7.39 mm
- net Net-(J104-Pin_1): track 0.00 -> 6.52 mm
- net /RG2: track 0.00 -> 6.39 mm
- net /RightLegDrive: track 0.00 -> 5.72 mm
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
Commit message: små ændringer med routing igen
Routing:
- net Net-(C101-Pad1): track 9.11 -> 1.14 mm
- net /HP+: track 29.4 -> 22.8 mm
Changed lines of the file:
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@@
-	)
-	(segment
-		(start 146.68238 101.31762)
-		(end 146.68238 105.5)
-		(width 0.2)
-		(layer "F.Cu")
-		(net 1)
-	)
-	(segment
-		(start 146.68238 101.31762)
-		(end 144 98.63524)
-		(width 0.2)
-		(layer "F.Cu")
-		(net 1)
 	)
 	(segment
@@
 	)
 	(segment
-		(start 143 94.5)
-		(end 141.5 96)
-		(width 0.2)
-		(layer "F.Cu")
-		(net 35)
-	)
-	(segment
-		(start 141.5 105.5)
+		(start 141 104)
+		(end 145 100)
+		(width 0.2)
+		(layer "F.Cu")
+		(net 35)
+	)
+	(segment
+		(start 141 106)
 		(end 139 108)
 		(width 0.2)
@@
 	)
 	(segment
-		(start 145 94.5)
-		(end 143 94.5)
+		(start 146.5 99.5)
+		(end 146.5 97.5)
+		(width 0.2)
+		(layer "F.Cu")
+		(net 35)
+	)
+	(segment
+		(start 141 106)
+		(end 141 104)
 		(width 0.2)
 		(layer "F.Cu")
@@
 	)
 	(segment
-		(start 141.5 96)
-		(end 141.5 105.5)
-		(width 0.2)
-		(layer "F.Cu")
-		(net 35)
-	)
-	(segment
-		(start 146.5 97.5)
-		(end 146.5 96)
-		(width 0.2)
-		(layer "F.Cu")
-		(net 35)
-	)
-	(segment
-		(start 146.5 96)
-		(end 145 94.5)
+		(start 146 100)
+		(end 146.5 99.5)
 		(width 0.2)
 		(layer "F.Cu")
@@
 		(width 0.2)
 		(layer "F.Cu")
+		(net 35)
+	)
+	(segment
+		(start 145 100)
+		(end 146 100)
+		(width 0.2)
+		(layer "F.Cu")

Commit message: routed pcb
Parts:
- removed J110, J111, J113: Conn_01x06_Pin, Connector_PinHeader_2.54mm:PinHeader_1x06_P2.54mm_Vertical
- removed TP120, TP121: TestPoint, TestPoint:TestPoint_Pad_D3.0mm
- added D101: LED, LED_THT:LED_D5.0mm, F.Cu at (184.5, 70.0)
- added J105: Conn_02x06_Odd_Even, Connector_PinHeader_2.54mm:PinHeader_2x06_P2.54mm_Vertical, F.Cu at (195.0, 93.7)
- added JP101: Jumper_2_Small_Bridged, Connector_PinHeader_2.54mm:PinHeader_1x02_P2.54mm_Vertical, F.Cu at (151.1, 72.6)
- added R116: 470, Resistor_THT:R_Axial_DIN0207_L6.3mm_D2.5mm_P10.16mm_Horizontal, F.Cu at (190.5, 76.2)
- moved R101 28.9 mm to (143.3, 78.0), turned to 180 degrees
- moved J104 17.0 mm to (166.0, 131.0)
- moved C103 8.75 mm to (125.7, 78.0), turned to 0 degrees
- moved L101 5.45 mm to (144.6, 72.5)
- moved C110 3.05 mm to (184.4, 91.1)
- moved C111 3.05 mm to (187.6, 91.1)
- moved R104 1.00 mm to (117.6, 116.0)
- moved R105 1.00 mm to (107.4, 119.0)
- moved C101 0.39 mm to (146.5, 105.2)
- moved C109 0.29 mm to (138.9, 98.7)
Connections:
- J104 pad 1: Net-(J104-Pin_1) -> /R_LEG
- J104 pad 2: /R_LEG -> Net-(J104-Pin_2)
- J112 pad 1: /SIGNAL_OUT -> /GAIN_BLOCK_OUT
- J112 pad 6: /SIGNAL_AMP -> /ADC_IN
- L101 pad 1: /5V_USB -> Net-(JP101-B)
- R108 pad 2: Net-(J104-Pin_1) -> Net-(J104-Pin_2)
- U102 pad 10: Net-(J104-Pin_1) -> Net-(J104-Pin_2)
- U102 pad 8: Net-(J104-Pin_1) -> Net-(J104-Pin_2)
Routing:
- net /R_LEG: track 31.0 -> 135.2 mm
- net /RightLegDrive: track 5.72 -> 92.4 mm
- net /V-IN: track 4.34 -> 64.3 mm
- net /ADC_IN: track 14.1 -> 66.6 mm
- net /V+IN: track 3.71 -> 55.2 mm
- net /LP_IN: track 5.42 -> 53.3 mm
- net /HP+: track 22.8 -> 67.1 mm, vias 0 -> 1
- net /HP_OUT: track 10.3 -> 51.1 mm, vias 0 -> 1
- net /INA_OUT: track 0.00 -> 39.9 mm
- net Net-(J104-Pin_2): track 0.00 -> 38.3 mm
- net /LP+: track 7.39 -> 43.9 mm
- net /L_ARM: track 25.7 -> 51.8 mm
- net +5V: track 0.00 -> 20.9 mm
- net /GAIN_BLOCK_OUT: track 16.1 -> 35.7 mm
- net /VGND: track 134.2 -> 118.0 mm
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Other:
- board text added: "ADC_IN"
- board text added: "EKG Print Gruppe ST7 AU 3. Semester December 2025 V1.0"
- board text added: "GAIN_O"
- board text added: "R_L_D"
- board text removed: "SIG_O"
